File: kicad/ULX4M-PCIe-IO_x4_half.kicad_pcb (KiCad board)
At the start: 4 copper layers, 167.7 x 111.2 mm, 255 parts, among them J1 PCIexpress_bracket, J10 FCR684205R, J11 OLED, J12 641737-1, J13 39-30-0060, J14 LM7805_EN, J15 POE, J16 Barrel_Jack, J17 JTAG, J18 I2C_to_ID, J19 PCIe_JTAG, J2 PCIexpress_x4, J20 PCIe_I2C, J21 PCIe_1X_4X, J3 SFP+, J4 SFP+, J5 HAT, J6 EXT_USB, J7 Micro_SD_Card_CD, J8 Board_To_Board, J9 FCR684205T, P1 GPDI0, SW1 SW_DIP_x08, SW2 SW_DIP_x08, U1 TPD4E02B04DQA, U10 TPD4E02B04DQA, U11 TPD4E02B04DQA, U12 TPD4E02B04DQA, U13 AT24CS32-SSHM, U14 LM78M05_TO252, U2 TPD4E02B04DQA, U3 TPD4E02B04DQA, U4 TPD4E02B04DQA, U5 TPD4E02B04DQA, U6 TPD4E02B04DQA, U7 TPD4E02B04DQA, U8 TPD4E02B04DQA, U9 TPD4E02B04DQA

Commit message: Routing
Routing:
- net OLED_CLK: track 69.9 -> 113.9 mm, vias 2 -> 3
- net OLED_MOSI: track 69.7 -> 110.8 mm, vias 2 -> 3
- net OLED_RES: track 69.5 -> 107.5 mm, vias 2 -> 3
- net OLED_DC: track 70.3 -> 101.8 mm, vias 2 -> 3
- net /RX_LOS_1: track 73.0 -> 104.2 mm
- net RS1: track 73.7 -> 104.6 mm
- net RS0: track 72.1 -> 102.0 mm
- net SFP1_MOD_ABS: track 110.0 -> 124.5 mm
- net SFP0_MOD_ABS: track 106.8 -> 116.8 mm
- net GND: track 116.3 -> 121.9 mm, vias 140 -> 141
- net /TX_FAULT_1: track 105.3 -> 104.0 mm

Commit message: Routing
Routing:
- net OLED_BL: track 55.0 -> 84.7 mm
- net OLED_CS: track 52.6 -> 67.9 mm
- net GND: track 121.9 -> 123.3 mm, vias 141 -> 143
- net +5V: track 427.7 -> 426.6 mm

Commit message: Routing
Parts:
- moved U11 117.9 mm to (278.8, 204.0)
- moved U12 115.1 mm to (269.9, 204.3)
Routing:
- net RS1: track 104.6 -> 130.1 mm
- net SFP1_MOD_ABS: track 124.5 -> 142.1 mm
- net SDA0: track 233.8 -> 251.3 mm
- net SCL0: track 239.3 -> 255.5 mm
- net +3.3V: track 542.8 -> 548.7 mm, vias 26 -> 28
